Commit message: When I fixed the robot joint angles, I did not think to flip the joint limits as well.

File: motoman_es_support/urdf/es200rn_120_macro.xacro (robot description, xacro)
@@ -174,5 +174,5 @@
       <child link="${prefix}link_u"/>
       <axis xyz="0 -1 0"/>
-      <limit lower="${radians(-138.0)}" upper="${radians(78.0)}" effort="0" velocity="${radians(85)}"/>
+      <limit lower="${radians(-78.0)}" upper="${radians(138.0)}" effort="0" velocity="${radians(85)}"/>
     </joint>
     <joint name="${prefix}joint_r" type="revolute">

Commit message: Constrained robot base axis to -100 degrees

File: motoman_es_support/urdf/es200rn_120_macro.xacro (robot description, xacro)
@@ -160,5 +160,5 @@
       <child link="${prefix}link_s"/>
       <axis xyz="0 0 1"/>
-      <limit lower="${radians(-180)}" upper="${radians(180)}" effort="0" velocity="${radians(90)}"/>
+      <limit lower="${radians(-100)}" upper="${radians(180)}" effort="0" velocity="${radians(90)}"/>
     </joint>
     <joint name="${prefix}joint_l" type="revolute">
